File: battery_switch/battery_switch.kicad_pcb (KiCad board)
At the start: 2 copper layers, 51.1 x 53 mm, 36 parts, among them J1 Conn_01x08, J5 Conn_01x02, J6 Conn_01x02, J7 Conn_01x02, J9 Conn_01x02, Q1 SUD50P04-08, Q2 SUD50P04-08, Q3 SUD50P04-08, Q4 SUD50P04-08, Q5 SUD50P04-08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

Commit message: completed layout
Parts:
- added REF**: MountingHole_2.7mm_M2.5, Mounting_Holes:MountingHole_2.7mm_M2.5, F.Cu at (177.5, 119.9)
- added REF**: MountingHole_2.7mm_M2.5, Mounting_Holes:MountingHole_2.7mm_M2.5, F.Cu at (132.3, 119.9)
- added REF**: MountingHole_2.7mm_M2.5, Mounting_Holes:MountingHole_2.7mm_M2.5, F.Cu at (132.3, 67.1)
- added REF**: MountingHole_2.7mm_M2.5, Mounting_Holes:MountingHole_2.7mm_M2.5, F.Cu at (177.5, 67.1)
Routing:
- net Net-(Q5-Pad1): track 11.8 -> 58.5 mm, vias 2 -> 4
- net Net-(D1-Pad1): track 4.17 -> 49.8 mm
- net Net-(C7-Pad1): track 9.69 -> 51.6 mm, vias 0 -> 2
- net Net-(Q3-Pad1): track 11.3 -> 42.6 mm, vias 2 -> 4
- net Net-(C8-Pad1): track 10.7 -> 40.9 mm, vias 0 -> 2
- net Net-(C9-Pad1): track 9.69 -> 36.2 mm
- net /~VALID1: track 37.3 -> 36.5 mm
- net /EN: track 27.9 -> 27.4 mm
Other:
- board size 51.1 x 53 mm -> 51.1 x 58.7 mm
- board text added: "'18 CC BY 4.0"
- board text added: "Triple Hot Swap Switch by Nirav Patel http://eclecti.cc"
